Commit message: update diffbot urdf and add nav2 param config

File: ros2_ws/install/polaris_controller/share/polaris_controller/urdf/diffbot.urdf.xacro (robot description, xacro)
@@ -4,9 +4,10 @@
   <xacro:arg name="prefix" default="" />
   <xacro:arg name="use_mock_hardware" default="false" />
+  <!-- <xacro:include filename="$(find my_diff_drive_bot)/description/robot.urdf.xacro" /> -->
   <xacro:include filename="$(find ros2_control_demo_description)/diffbot/urdf/diffbot_description.urdf.xacro" />
   <!-- Import Rviz colors -->
   <xacro:include filename="$(find ros2_control_demo_description)/diffbot/urdf/diffbot.materials.xacro" />
   <!-- Import diffbot ros2_control description -->
-  <xacro:include filename="$(find polaris_controller)/ros2_control/diffbot.ros2_control.xacro" />
+  <xacro:include filename="$(find polaris_controller)/ros2_control/robot.ros2_control.xacro" />
   <xacro:diffbot prefix="$(arg prefix)" />
   <xacro:diffbot_ros2_control

File: ros2_ws/install/ros2_control_demo_description/share/ros2_control_demo_description/diffbot/urdf/diffbot_description.urdf.xacro (robot description, xacro)
@@ -1,163 +1,178 @@
 <?xml version="1.0"?>
 <robot xmlns:xacro="http://www.ros.org/wiki/xacro">
+  <xacro:include filename="inertial_macros.xacro"/>
   <xacro:macro name="diffbot" params="prefix">
-  <!-- Constants for robot dimensions -->
-  <xacro:property name="PI" value="3.1415926535897931"/>
-  <xacro:property name="base_mass" value="0.3" /> <!-- arbitrary value for base mass -->
-  <xacro:property name="base_width" value="0.1" />
-  <xacro:property name="base_length" value="0.1" />
-  <xacro:property name="base_height" value="0.05" />
-  <xacro:property name="wheel_mass" value="0.3" /> <!-- arbitrary value for wheel mass -->
-  <xacro:property name="wheel_len" value="0.020" />
-  <xacro:property name="wheel_radius" value="0.015" />
-  <xacro:property name="caster_wheel_mass" value="0.1" /> <!-- arbitrary value for caster wheel mass -->
-  <xacro:property name="caster_wheel_radius" value="0.015" />
-  <xacro:property name="z_offset" value="-${base_height/2}" /> <!-- Space btw top of beam and the each joint -->
   <!-- Base Link -->
   <link name="${prefix}base_link">
+  </link>
+   <!-- CHASSIS LINK -->
+  <joint name="${prefix}chassis_joint" type="fixed">
+    <parent link="${prefix}base_link"/>
+    <child link="${prefix}chassis"/>
+    <origin xyz="-0.452 0 0"/>
+</joint>
+<link name="${prefix}chassis">
+    <visual>
+        <origin xyz="0.272 0 0.016"/>
+        <geometry>
+            <mesh filename="file://$(find my_diff_drive_bot)/meshes/chassis_link.stl" scale="0.001 0.001 0.001"/>
+        </geometry>
+        <material name="silver"/>
+    </visual>
     <collision>
+        <origin xyz="0.272 0 0.016"/>
+        <geometry>
+            <mesh filename="file://$(find my_diff_drive_bot)/meshes/chassis_link.stl" scale="0.001 0.001 0.001"/>
+        </geometry>
+        <material name="silver"/>
+    </collision>
+    <xacro:inertial_box mass="10.0" x="0.544" y="0.422" z="0.656">
+        <origin xyz="0.272 0 0.328" rpy="0 0 0"/>
+    </xacro:inertial_box>
+</link>
+<!-- LEFT WHEEL LINK -->
+<joint name="${prefix}left_wheel_joint" type="continuous">
+  <parent link="${prefix}base_link"/>
+  <child link="${prefix}left_wheel"/>
+  <origin xyz="0 0.148 0" rpy="-${pi/2} 0 0"/>
+  <axis xyz="0 0 1"/>
+</joint>
+<link name="${prefix}left_wheel">
+  <visual>
+      <geometry>
+          <cylinder radius="0.0625" length="0.023"/>
+      </geometry>
+      <materaial name="black"/>
+  </visual>
+  <collision>
+      <geometry>
+          <cylinder radius="0.0625" length="0.023"/>
+      </geometry>
+      <materaial name="black"/>
+  </collision>
+  <xacro:inertial_cylinder mass="0.15" length="0.023" radius="0.0625">
       <origin xyz="0 0 0" rpy="0 0 0"/>
+  </xacro:inertial_cylinder>
+</link>
+ <!-- LEFT CASTER WHEEL LINK -->
+ <joint name="${prefix}left_caster_joint" type="continuous">
+  <parent link="${prefix}base_link"/>
+  <child link="${prefix}left_caster_link"/>
+  <origin xyz="-0.420 0.139 0.007" rpy="-${pi} 0 0"/>
+  <axis xyz="0 0 1"/>
+</joint>
+<link name="${prefix}left_caster_link">
+  <materaial name="black"/>
+  <visual>
+      <origin xyz="0 0 0" rpy="-${pi} 0 0"/>
       <geometry>
-        <box size="${base_width} ${base_length} ${base_height}"/>
+          <mesh filename="file://$(find my_diff_drive_bot)/meshes/caster_link.stl" scale="0.001 0.001 0.001"/>
       </geometry>
-    </collision>
-    <visual>
-      <origin xyz="0 0 ${base_height/2}" rpy="0 0 0"/>
+  </visual>
+  <collision>
+      <origin xyz="0 0 0" rpy="-${pi} 0 0"/>
       <geometry>
-        <box size="${base_width} ${base_length} ${base_height}"/>
+          <mesh filename="file://$(find my_diff_drive_bot)/meshes/caster_link.stl" scale="0.001 0.001 0.001"/>
       </geometry>
-      <material name="orange"/>
-    </visual>
-    <inertial>
+      <materaial name="black"/>
+  </collision>
+  <xacro:inertial_cylinder mass="0.1" length="0.090" radius="0.03">
       <origin xyz="0 0 0" rpy="0 0 0"/>
-      <mass value="${base_mass}"/>
-      <inertia
-        ixx="${base_mass / 12.0 * (base_length*base_length + base_height*base_height)}" ixy="0.0" ixz="0.0"
-        iyy="${base_mass / 12.0 * (base_height*base_height + base_width*base_width)}" iyz="0.0"
-        izz="${base_mass / 12.0 * (base_width*base_width + base_length*base_length)}"/>
-      </inertial>
-    </link>
-    <joint name="${prefix}left_wheel_joint" type="continuous">
-      <parent link="${prefix}base_link"/>
-      <child link="${prefix}left_wheel"/>
-      <origin xyz="0 -${base_width/2} ${z_offset}" rpy="0 0 0"/>
-      <axis xyz="0 1 0"/>
-      <dynamics damping="0.2"/>
-      <limit effort="100" velocity="1.0"/>
-    </joint>
-    <!-- left wheel Link -->
-    <link name="${prefix}left_wheel">
-      <collision>
-        <origin xyz="0 0 0" rpy="${PI/2} 0 0"/>
-        <geometry>
-          <cylinder length="${wheel_len}" radius="${wheel_radius}"/>
-        </geometry>
-      </collision>
-      <visual>
-        <origin xyz="0 0 0" rpy="${PI/2} 0 0"/>
-        <geometry>
-          <cylinder length="${wheel_len}" radius="${wheel_radius}"/>
-        </geometry>
-        <material name="black"/>
-      </visual>
-      <inertial>
-        <origin xyz="0 0 0" rpy="${PI/2} 0 0"/>
-        <mass value="${wheel_mass}"/>
-        <inertia
-          ixx="${wheel_mass / 12.0 * (3*wheel_radius*wheel_radius + wheel_len*wheel_len)}" ixy="0.0" ixz="0.0"
-          iyy="${wheel_mass / 12.0 * (3*wheel_radius*wheel_radius + wheel_len*wheel_len)}" iyz="0.0"
-          izz="${wheel_mass / 2.0 * wheel_radius*wheel_radius}"/>
-        </inertial>
-      </link>
-    <joint name="${prefix}right_wheel_joint" type="continuous">
-      <parent link="${prefix}base_link"/>
-      <child link="${prefix}right_wheel"/>
-      <origin xyz="0 ${base_width/2} ${z_offset}" rpy="0 0 0"/>
-      <axis xyz="0 1 0"/>
-      <dynamics damping="0.2"/>
-      <limit effort="100" velocity="1.0"/>
-    </joint>
-    <!-- right wheel Link -->
-    <link name="${prefix}right_wheel">
-      <collision>
-        <origin xyz="0 0 0" rpy="${PI/2} 0 0"/>
-        <geometry>
-          <cylinder length="${wheel_len}" radius="${wheel_radius}"/>
-        </geometry>
-      </collision>
-      <visual>
-        <origin xyz="0 0 0" rpy="${PI/2} 0 0"/>
-        <geometry>
-          <cylinder length="${wheel_len}" radius="${wheel_radius}"/>
-        </geometry>
-        <material name="black"/>
-      </visual>
-      <inertial>
-        <origin xyz="0 0 0" rpy="${PI/2} 0 0"/>
-        <mass value="${wheel_mass}"/>
-        <inertia
-          ixx="${wheel_mass / 12.0 * (3*wheel_radius*wheel_radius + wheel_len*wheel_len)}" ixy="0.0" ixz="0.0"
-          iyy="${wheel_mass / 12.0 * (3*wheel_radius*wheel_radius + wheel_len*wheel_len)}" iyz="0.0"
-          izz="${wheel_mass / 2.0 * wheel_radius*wheel_radius}"/>
-        </inertial>
-      </link>
-    <joint name="${prefix}caster_frontal_wheel_joint" type="fixed">
-      <parent link="${prefix}base_link"/>
-      <child link="${prefix}caster_frontal_wheel"/>
-      <origin xyz="${base_width/2 - caster_wheel_radius} 0 ${z_offset}" rpy="0 0 0"/>
-    </joint>
-    <!-- caster frontal wheel Link -->
-    <link name="${prefix}caster_frontal_wheel">
-      <collision>
-        <origin xyz="0 0 0" rpy="0 0 0"/>
-        <geometry>
-          <sphere radius="${caster_wheel_radius}"/>
-        </geometry>
-      </collision>
-      <visual>
-        <origin xyz="0 0 0" rpy="0 0 0"/>
-        <geometry>
-          <sphere radius="${caster_wheel_radius}"/>
-        </geometry>
-        <material name="white"/>
-      </visual>
-      <inertial>
-        <origin xyz="0 0 0" rpy="0 0 0"/>
-        <mass value="${caster_wheel_mass}"/>
-        <inertia
-          ixx="${caster_wheel_mass * 0.4 * (caster_wheel_radius * caster_wheel_radius)}" ixy="0.0" ixz="0.0"
-          iyy="${caster_wheel_mass * 0.4 * (caster_wheel_radius * caster_wheel_radius)}" iyz="0.0"
-          izz="${caster_wheel_mass * 0.4 * (caster_wheel_radius * caster_wheel_radius)}"/>
-        </inertial>
-      </link>
-    <joint name="${prefix}caster_rear_wheel_joint" type="fixed">
-      <parent link="${prefix}base_link"/>
-      <child link="${prefix}caster_rear_wheel"/>
-      <origin xyz="${-base_width/2 + caster_wheel_radius} 0 ${z_offset}" rpy="0 0 0"/>
-    </joint>
-    <!-- caster rear wheel Link -->
-    <link name="${prefix}caster_rear_wheel">
-      <collision>
-        <origin xyz="0 0 0" rpy="0 0 0"/>
-        <geometry>
-          <sphere radius="${caster_wheel_radius}"/>
-        </geometry>
-      </collision>
-      <visual>
-        <origin xyz="0 0 0" rpy="0 0 0"/>
-        <geometry>
-          <sphere radius="${caster_wheel_radius}"/>
-        </geometry>
-        <material name="white"/>
-      </visual>
-      <inertial>
-        <origin xyz="0 0 0" rpy="0 0 0"/>
-        <mass value="${caster_wheel_mass}"/>
-        <inertia
-          ixx="${caster_wheel_mass * 0.4 * (caster_wheel_radius * caster_wheel_radius)}" ixy="0.0" ixz="0.0"
-          iyy="${caster_wheel_mass * 0.4 * (caster_wheel_radius * caster_wheel_radius)}" iyz="0.0"
-          izz="${caster_wheel_mass * 0.4 * (caster_wheel_radius * caster_wheel_radius)}"/>
-        </inertial>
-      </link>
+  </xacro:inertial_cylinder>
+</link>
+<!-- LEFT CASTER WHEEL -->
+<joint name="${prefix}left_caster_wheel_joint" type="continuous">
+  <parent link="${prefix}left_caster_link"/>
+  <child link="${prefix}left_caster_wheel"/>
+  <origin xyz="0.02 0 0.04" rpy="-${pi/2} 0 0"/>
+  <axis xyz="0 0 1"/>
+</joint>
+<link name="${prefix}left_caster_wheel">
+  <visual>
+      <geometry>
+          <cylinder radius="0.025" length="0.018"/>
+      </geometry>
+  </visual>
+  <collision>
+      <geometry>
+          <cylinder radius="0.025" length="0.018"/>
+      </geometry>
+  </collision>
+  <xacro:inertial_cylinder mass="0.1" length="0.018" radius="0.025">
+      <origin xyz="0 0 0" rpy="0 0 0"/>
+  </xacro:inertial_cylinder>
+</link>
+<!-- RIGHT WHEEL LINK -->
+<joint name="${prefix}right_wheel_joint" type="continuous">
+  <parent link="${prefix}base_link"/>
+  <child link="${prefix}right_wheel"/>
+  <origin xyz="0 -0.148 0" rpy="${pi/2} 0 0"/>
+  <axis xyz="0 0 -1"/>
+</joint>
+<link name="${prefix}right_wheel">
+  <visual>
+      <geometry>
+          <cylinder radius="0.0625" length="0.023"/>
+      </geometry>
+      <materaial name="black"/>
+  </visual>
+  <collision>
+      <geometry>
+          <cylinder radius="0.0625" length="0.023"/>
+      </geometry>
+      <materaial name="black"/>
+  </collision>
+  <xacro:inertial_cylinder mass="0.15" length="0.023" radius="0.0625">
+      <origin xyz="0 0 0" rpy="0 0 0"/>
+  </xacro:inertial_cylinder>
+</link>
+<!-- RIGHT CASTER WHEEL LINK -->
+<joint name="${prefix}right_caster_joint" type="continuous">
+  <parent link="${prefix}base_link"/>
+  <child link="${prefix}right_caster_link"/>
+  <origin xyz="-0.420 -0.139 0.007" rpy="-${pi} 0 0"/>
+  <axis xyz="0 0 1"/>
+</joint>
+<link name="${prefix}right_caster_link">
+  <materaial name="black"/>
+  <visual>
+      <origin xyz="0 0 0" rpy="-${pi} 0 0"/>
+      <geometry>
+          <mesh filename="file://$(find my_diff_drive_bot)/meshes/caster_link.stl" scale="0.001 0.001 0.001"/>
+      </geometry>
+  </visual>
+  <collision>
+      <origin xyz="0 0 0" rpy="-${pi} 0 0"/>
+      <geometry>
+          <mesh filename="file://$(find my_diff_drive_bot)/meshes/caster_link.stl" scale="0.001 0.001 0.001"/>
+      </geometry>
+      <materaial name="black"/>
+  </collision>
+  <xacro:inertial_cylinder mass="0.1" length="0.090" radius="0.03">
+      <origin xyz="0 0 0" rpy="0 0 0"/>
+  </xacro:inertial_cylinder>
+</link>
+<!-- RIGHT CASTER WHEEL -->
+<joint name="${prefix}right_caster_wheel_joint" type="continuous">
+  <parent link="${prefix}right_caster_link"/>
+  <child link="${prefix}right_caster_wheel"/>
+  <origin xyz="0.02 0 0.04" rpy="-${pi/2} 0 0"/>
+  <axis xyz="0 0 1"/>
+</joint>
+<link name="${prefix}right_caster_wheel">
+  <visual>
+      <geometry>
+          <cylinder radius="0.025" length="0.018"/>
+      </geometry>
+  </visual>
+  <collision>
+      <geometry>
+          <cylinder radius="0.025" length="0.018"/>
+      </geometry>
+  </collision>
+  <xacro:inertial_cylinder mass="0.1" length="0.018" radius="0.025">
+      <origin xyz="0 0 0" rpy="0 0 0"/>
+  </xacro:inertial_cylinder>
+</link>
   </xacro:macro>
 </robot>
